Commit message: added sonars

File: environment_pkg/urdf/base.urdf.xacro (robot description, xacro)
@@ -99,4 +99,14 @@
     <xacro:caster side="back_right"  radius="${caster_radius}" width="${caster_width}" separation_x="${-caster_separation_x}" separation_y="${ caster_separation_y}" offset_x="${caster_offset_x}" offset_y="${caster_offset_y}" offset_z="${caster_offset_z}" parent="${name}"/>
     <xacro:caster side="back_left"   radius="${caster_radius}" width="${caster_width}" separation_x="${-caster_separation_x}" separation_y="${-caster_separation_y}" offset_x="${caster_offset_x}" offset_y="${caster_offset_y}" offset_z="${caster_offset_z}" parent="${name}"/>
+    <!--Sonar base-->
+    <xacro:sonar_sensor name="${name}_sonar1" parent="${name}_link" ros_topic="${name}_sonar1" update_rate="10.0" min_range="0.2" max_range="3.5" field_of_view="0.785398" ray_count="5">
+      <origin xyz="0.0 0.0 0.0" rpy="0 0 0"/>
+    </xacro:sonar_sensor>
+    <xacro:sonar_sensor name="${name}_sonar2" parent="${name}_link" ros_topic="${name}_sonar2" update_rate="10.0" min_range="-0.2" max_range="-3.5" field_of_view="0.785398" ray_count="5">
+      <origin xyz="0.0 0.0 0.0" rpy="0 0 0"/>
+    </xacro:sonar_sensor>
+    <xacro:sonar_sensor name="${name}_sonar3" parent="${name}_link" ros_topic="${name}_sonar3" update_rate="10.0" min_range="0.2" max_range="3.5" field_of_view="0.785398" ray_count="5">
+      <origin xyz="0.0 0.0 0.0" rpy="0 0 0"/>
+    </xacro:sonar_sensor>
   </xacro:macro>
 </robot>

File: environment_pkg/urdf/base_sensors.urdf.xacro (robot description, xacro)
@@ -16,5 +16,5 @@
   <xacro:arg name="y" default="0"/>
   <xacro:arg name="yaw" default="0"/>
-  <xacro:include filename="$(find environment_pkg)/urdf/tiago/base.urdf.xacro"/>
+  <xacro:include filename="$(find environment_pkg)/urdf/base.urdf.xacro"/>
   <xacro:include filename="$(find pmb2_description)/urdf/sensors/hokuyo_urg_04lx_ug01_laser.urdf.xacro"/>
   <xacro:include filename="$(find pmb2_description)/urdf/sensors/sick_tim551_laser.urdf.xacro"/>

File: environment_pkg/urdf/tiago.urdf.xacro (robot description, xacro)
@@ -1,5 +1,5 @@
 <?xml version="1.0"?>
 <!--
-  Copyright (c) 2022 PAL Robotics S.L. All rights reserved.
+  Copyright (c) 2021 PAL Robotics S.L. All rights reserved.
   Licensed under the Apache License, Version 2.0 (the "License");
   you may not use this file except in compliance with the License.
@@ -11,24 +11,21 @@
   See the License for the specific language governing permissions and
   limitations under the License.
- -->
+-->
 <robot  xmlns:xacro="http://ros.org/wiki/xacro"
         name="tiago" >
-    <xacro:arg name="arm" default="right-arm"/> <!-- right-arm, no-arm -->
+    <xacro:arg name="arm" default="true"/> <!-- true, false -->
     <xacro:arg name="wrist_model" default="wrist-2010"/>
-    <xacro:arg name="end_effector" default="pal-hey5"/> <!-- no-end-effector, pal-gripper, pal-hey5-->
-    <xacro:arg name="ft_sensor" default="schunk-ft"/> <!-- no-ft-sensor, schunk-ft -->
-    <xacro:arg name="laser_model" default="sick-571"/> <!-- no-laser, hokuyo, sick-551, sick-561, sick-571-->
-    <xacro:arg name="camera_model" default="orbbec-astra"/> <!-- no-camera, orbbec-astra, orbbec-astra-pro, asus-xtion -->
+    <xacro:arg name="end_effector" default="pal-hey5"/> <!-- false, pal-gripper, pal-hey5, schunk-wsg-->
+    <xacro:arg name="ft_sensor" default="schunk-ft"/> <!-- false, schunk-ft -->
+    <xacro:arg name="laser_model" default="sick-571"/> <!-- false, hokuyo, sick-551, sick-561, sick-571-->
+    <xacro:arg name="camera_model" default="orbbec-astra"/> <!-- false, orbbec-astra, orbbec-astra-pro, asus-xtion -->
     <xacro:arg name="has_thermal_camera" default="false"/>
     <xacro:arg name="multiple" default="false"/>
-    <xacro:arg name="description_calibration_dir" default="$(find tiago_description)/urdf/calibration"/>
-    <xacro:arg name="extrinsic_calibration_dir" default="$(find tiago_description)/urdf/calibration"/>
+    <xacro:arg name="description_calibration_dir" default="$(find tiago_description_calibration)/urdf/calibration"/>
+    <xacro:arg name="extrinsic_calibration_dir" default="$(find tiago_description_calibration)/urdf/calibration"/>
     <xacro:arg name="namespace" default=""/>
     <xacro:arg name="no_safety_eps" default="false"/>
-    <xacro:arg name="use_sim" default="false"/>
-    <xacro:property name="arm" value="$(arg arm)" />
-    <xacro:if value="${arm not in ['right-arm', 'no-arm']}">
-      <xacro:wrong_arm/>
-    </xacro:if>
+    <xacro:arg name="base_type" default="pmb2"/> <!-- pmb2, omni_base -->
+    <xacro:arg name="fixed_torso" default="false" />
     <xacro:property name="wrist_model" value="$(arg wrist_model)" />
     <xacro:property name="end_effector" value="$(arg end_effector)" />
@@ -38,27 +35,33 @@
     <xacro:property name="is_multiple" value="$(arg multiple)" />
     <xacro:property name="nsp" value="$(arg namespace)" />
+    <xacro:property name="base_type" value="$(arg base_type)" />
     <xacro:property name="no_safety_eps" value="$(arg no_safety_eps)" />
-    <xacro:property name="has_arm" value="${arm != 'no-arm'}"/>
-  <xacro:if value="${has_arm}">
+    <xacro:property name="fixed_torso" value="$(arg fixed_torso)" />
+  <xacro:if value="$(arg arm)">
     <xacro:if value="${wrist_model not in ['wrist-2010', 'wrist-2017']}">
       <xacro:wrong_wrist_model/>
     </xacro:if>
   </xacro:if>
-  <xacro:if value="${end_effector not in ['no-end-effector', 'pal-gripper', 'pal-hey5', 'custom']}">
+  <xacro:if value="${end_effector not in ['false', False, 'pal-gripper', 'pal-hey5', 'schunk-wsg', 'robotiq-2f-85', 'robotiq-2f-140', 'robotiq-epick', 'custom', 'no-ee']}">
     <xacro:wrong_end_effector/>
   </xacro:if>
-  <xacro:if value="${ft_sensor not in ['no-ft-sensor', 'schunk-ft']}">
+  <xacro:if value="${ft_sensor not in ['false', False, 'schunk-ft']}">
     <xacro:wrong_ft_sensor/>
   </xacro:if>
-  <xacro:if value="${laser_model not in ['no-laser', 'sick-551', 'sick-561', 'sick-571', 'hokuyo']}">
+  <xacro:if value="${laser_model not in ['false', False, 'sick-551', 'sick-561', 'sick-571', 'hokuyo', 'ydlidar-tg30', 'ydlidar-tg15']}">
     <xacro:wrong_laser_model/>
   </xacro:if>
-  <xacro:if value="${camera_model not in ['no-camera', 'orbbec-astra', 'orbbec-astra-pro', 'asus-xtion']}">
+  <xacro:if value="${camera_model not in ['false', False, 'orbbec-astra', 'orbbec-astra-pro', 'asus-xtion']}">
     <xacro:wrong_camera_model/>
+  </xacro:if>
+  <xacro:if value="${base_type not in ['pmb2', 'omni_base']}">
+    <xacro:wrong_base_type/>
   </xacro:if>
         <!-- The properties below are modified using empy http://www.alcyone.com/software/empy/
              from the create_robot.py tool. Handle them with care -->
+   <xacro:property name="has_arm"                 value="$(arg arm)"/>
    <xacro:property name="has_schunk_ft"           value="${ft_sensor == 'schunk-ft'}"/>
-   <xacro:property name="has_ft_sensor"           value="${has_arm and has_schunk_ft}"/> <!-- This should be OR'ed with other FT sensors-->
+   <xacro:property name="has_ft_sensor"           value="${has_schunk_ft}"/> <!-- This should be OR'ed with other FT sensors-->
+   <xacro:property name="has_end_effector"        value="${end_effector not in ['false', False, 'no-ee']}"/>
    <xacro:property name="end_effector_link"       value="${'wrist_ft_tool_link' if has_ft_sensor else 'arm_tool_link'}"/>
    <xacro:property name="end_effector_name"       value="${'hand' if end_effector == 'pal-hey5' else 'gripper'}"/>
@@ -66,6 +69,18 @@
    <xacro:property name="description_calibration_dir"       value="${arg description_calibration_dir}"/>
   <!-- The following included files set up definitions of parts of the robot body -->
+  <!--File includes-->
+  <xacro:include filename="$(find pal_urdf_utils)/urdf/deg_to_rad.xacro" />
   <!-- Base -->
-  <xacro:include filename="$(find environment_pkg)/urdf/tiago/base_sensors.urdf.xacro" />
+  <xacro:include filename="$(find ${base_type}_description)/urdf/base/base_sensors.urdf.xacro" />
+  <xacro:include filename="$(find hector_sensors_description)/urdf/sonar_sensor.urdf.xacro"/>
+  <xacro:sonar_sensor name="base_sonar1" parent="base_link" ros_topic="base_sonar1" update_rate="10.0" min_range="0.2" max_range="3.5" field_of_view="0.785398" ray_count="5">
+    <origin xyz="0.0 0.0 0.0" rpy="0 0 0"/>
+  </xacro:sonar_sensor>
+  <xacro:sonar_sensor name="base_sonar2" parent="base_link" ros_topic="base_sonar2" update_rate="10.0" min_range="-0.2" max_range="-3.5" field_of_view="0.785398" ray_count="5">
+    <origin xyz="0.0 0.0 0.0" rpy="0 0 0"/>
+  </xacro:sonar_sensor>
+  <xacro:sonar_sensor name="base_sonar3" parent="base_link" ros_topic="base_sonar3" update_rate="10.0" min_range="0.2" max_range="3.5" field_of_view="0.785398" ray_count="5">
+    <origin xyz="0.0 0.0 0.0" rpy="0 0 0"/>
+  </xacro:sonar_sensor>
   <!-- Torso -->
   <xacro:include filename="$(find tiago_description)/urdf/torso/torso.urdf.xacro" />
@@ -74,23 +89,23 @@
     <xacro:include filename="$(find tiago_description)/urdf/arm/arm.urdf.xacro" />
     <xacro:include filename="$(find tiago_description)/urdf/end_effector/end_effector.urdf.xacro" />
-    <xacro:include filename="$(arg description_calibration_dir)/calibration_constants.urdf.xacro" />
+  <xacro:include filename="$(arg description_calibration_dir)/calibration_constants.urdf.xacro" />
   </xacro:if>
   <!-- Force Torque sensor -->
   <xacro:if value="${has_ft_sensor}">
     <xacro:include filename="$(find tiago_description)/urdf/sensors/ftsensor.urdf.xacro" />
-    <xacro:include filename="$(find tiago_description)/urdf/sensors/ftsensor.gazebo.xacro" />
   </xacro:if>
   <!-- Head -->
   <xacro:include filename="$(find tiago_description)/urdf/head/head.urdf.xacro" />
+  <!-- Materials for visualization -->
+  <xacro:include filename="$(find pal_urdf_utils)/urdf/materials.urdf.xacro" />
   <!-- Generic simulator_gazebo plugins -->
   <xacro:include filename="$(find tiago_description)/gazebo/gazebo.urdf.xacro" />
-  <!-- ros2_control -->
-  <xacro:include filename="$(find tiago_description)/ros2_control/ros2_control.urdf.xacro" />
-  <xacro:tiago_ros2_control
-    use_sim="$(arg use_sim)" />
-  <!-- Materials for visualization -->
-  <xacro:include filename="$(find pal_urdf_utils)/urdf/materials.urdf.xacro" />
   <!-- Now we can start using the macros included above to define the actual robot -->
-  <xacro:base_sensors name="base" laser_model="$(arg laser_model)" sonars="true" microphone="true"/>
+  <xacro:if value="${base_type == 'pmb2'}">
+    <xacro:base_sensors name="base" laser_model="$(arg laser_model)" sonars="true" microphone="true"/>
+  </xacro:if>
+  <xacro:if value="${base_type == 'omni_base'}">
+    <xacro:base_sensors name="base" front_laser_model="$(arg laser_model)" rear_laser_model="$(arg laser_model)"/>
+  </xacro:if>
   <xacro:tiago_torso name="torso" parent="base_link"/>
   <xacro:head name="head" parent="torso_lift_link" camera_model="$(arg camera_model)"
@@ -102,10 +117,9 @@
         <origin xyz="0.15505 0.014 -0.151" rpy="0 0 ${-90 * deg_to_rad}" />
       </xacro:tiago_arm>
-      <xacro:tiago_end_effector name="${end_effector_name}" parent="${end_effector_link}" type="${end_effector}" reflect="1"/>
-  </xacro:if>
+      <xacro:tiago_end_effector name="${end_effector_name}" parent="${end_effector_link}" type="${end_effector}" has_end_effector="${has_end_effector}" reflect="1"/>
   <!-- Force Torque sensor -->
   <xacro:if value="${has_ft_sensor}">
       <xacro:ft_sensor name="wrist" parent="arm_tool_link" />
-      <xacro:force_torque_sensor_gazebo name="wrist_ft" update_rate="100"/>
+  </xacro:if>
   </xacro:if>
   <!-- Thermal camera -->

Commit message: added sonars

File: environment_pkg/urdf/base.urdf.xacro (robot description, xacro)
@@ -100,5 +100,5 @@
     <xacro:caster side="back_left"   radius="${caster_radius}" width="${caster_width}" separation_x="${-caster_separation_x}" separation_y="${-caster_separation_y}" offset_x="${caster_offset_x}" offset_y="${caster_offset_y}" offset_z="${caster_offset_z}" parent="${name}"/>
     <!--Sonar base-->
-    <xacro:sonar_sensor name="${name}_sonar1" parent="${name}_link" ros_topic="${name}_sonar1" update_rate="10.0" min_range="0.2" max_range="3.5" field_of_view="0.785398" ray_count="5">
+    <!-- <xacro:sonar_sensor name="${name}_sonar1" parent="${name}_link" ros_topic="${name}_sonar1" update_rate="10.0" min_range="0.2" max_range="3.5" field_of_view="0.785398" ray_count="5">
       <origin xyz="0.0 0.0 0.0" rpy="0 0 0"/>
     </xacro:sonar_sensor>
@@ -108,5 +108,5 @@
     <xacro:sonar_sensor name="${name}_sonar3" parent="${name}_link" ros_topic="${name}_sonar3" update_rate="10.0" min_range="0.2" max_range="3.5" field_of_view="0.785398" ray_count="5">
       <origin xyz="0.0 0.0 0.0" rpy="0 0 0"/>
-    </xacro:sonar_sensor>
+    </xacro:sonar_sensor> -->
   </xacro:macro>
 </robot>

File: environment_pkg/urdf/base_sensors.urdf.xacro (robot description, xacro)
@@ -1,5 +1,5 @@
 <?xml version="1.0"?>
 <!--
-  Copyright (c) 2022 PAL Robotics S.L. All rights reserved.
+  Copyright (c) 2021 PAL Robotics S.L. All rights reserved.
   Licensed under the Apache License, Version 2.0 (the "License");
   you may not use this file except in compliance with the License.
@@ -11,14 +11,13 @@
   See the License for the specific language governing permissions and
   limitations under the License.
- -->
+-->
 <robot xmlns:xacro="http://ros.org/wiki/xacro">
-  <xacro:arg name="x" default="0"/>
-  <xacro:arg name="y" default="0"/>
-  <xacro:arg name="yaw" default="0"/>
-  <xacro:include filename="$(find environment_pkg)/urdf/base.urdf.xacro"/>
+  <xacro:include filename="$(find pmb2_description)/urdf/base/base.urdf.xacro"/>
   <xacro:include filename="$(find pmb2_description)/urdf/sensors/hokuyo_urg_04lx_ug01_laser.urdf.xacro"/>
   <xacro:include filename="$(find pmb2_description)/urdf/sensors/sick_tim551_laser.urdf.xacro"/>
   <xacro:include filename="$(find pmb2_description)/urdf/sensors/sick_tim561_laser.urdf.xacro"/>
   <xacro:include filename="$(find pmb2_description)/urdf/sensors/sick_tim571_laser.urdf.xacro"/>
+  <xacro:include filename="$(find pmb2_description)/urdf/sensors/ydlidar_tg30_laser.urdf.xacro"/>
+  <xacro:include filename="$(find pmb2_description)/urdf/sensors/ydlidar_tg15_laser.urdf.xacro"/>
   <xacro:include filename="$(find pmb2_description)/urdf/sensors/range.urdf.xacro"/>
   <xacro:include filename="$(find pmb2_description)/urdf/sensors/microphone.urdf.xacro"/>
@@ -29,4 +28,14 @@
   <!-- laser_model can be: false, hokuyo, sick-551, sick-561, sick-571-->
   <xacro:macro name="base_sensors" params=" name laser_model:=sick-571 sonars:=false microphone:=false ">
+    <xacro:if value="${laser_model == 'ydlidar-tg15' or laser_model == 'ydlidar-tg30'}">
+      <xacro:property name="base_laser_x" value="0.2095"/>
+      <xacro:property name="base_laser_y" value="0.0"/>
+      <xacro:property name="base_laser_z" value="0.00890"/>
+    </xacro:if>
+    <xacro:unless value="${laser_model == 'ydlidar-tg15' or laser_model == 'ydlidar-tg30'}">
+        <xacro:property name="base_laser_x" value="0.202"/>
+        <xacro:property name="base_laser_y" value="0.0"/>
+        <xacro:property name="base_laser_z" value="-0.004"/>
+    </xacro:unless>
     <xacro:if value="${laser_model == 'hokuyo'}">
       <!-- Laser -->
@@ -57,14 +66,55 @@
       </xacro:sick_tim571_laser>
     </xacro:if>
+    <xacro:if value="${laser_model == 'ydlidar-tg30'}">
+      <!-- Laser -->
+      <!-- Theoretic FOV = 360 -->
+      <xacro:ydlidar_tg30_laser name="${name}_laser" parent="${name}" ros_topic="scan_raw" update_rate="10" min_angle="${-65* deg_to_rad}" max_angle="${125 * deg_to_rad}" >
+        <origin xyz="${base_laser_x} ${base_laser_y} ${base_laser_z}" rpy="0 0 ${ -30 * deg_to_rad }" />
+      </xacro:ydlidar_tg30_laser>
+    </xacro:if>
+    <xacro:if value="${laser_model == 'ydlidar-tg15'}">
+      <!-- Laser -->
+      <!-- Theoretic FOV = 360 -->
+      <xacro:ydlidar_tg15_laser name="${name}_laser" parent="${name}" ros_topic="scan_raw" update_rate="10" min_angle="${-65 * deg_to_rad}" max_angle="${125 * deg_to_rad}" >
+        <origin xyz="${base_laser_x} ${base_laser_y} ${base_laser_z}" rpy="0 0 ${ -30 * deg_to_rad }" />
+      </xacro:ydlidar_tg15_laser>
+    </xacro:if>
     <xacro:if value="${sonars}">
       <!-- Sonars -->
-      <xacro:range_sensor name="${name}_sonar_03" parent="${name}" ros_topic="sonar_${name}" update_rate="5" maxRange="1.0" minRange="0.02" fov="0.5" radiation="ultrasound">
-        <origin xyz="-0.183 0.183 0.173" rpy="0 0 ${135 * deg_to_rad}"/>
+      <xacro:range_sensor name="${name}_sonar_01" parent="${name}" ros_topic="sonar4_${name}" update_rate="1" maxRange="3.0" minRange="0.02" fov="0.5" radiation="ultrasound">
+        <origin xyz="${0.259*cos(0*deg_to_rad)} ${0.259*sin(0*deg_to_rad)}  0.173" rpy="0 0 ${0*deg_to_rad}"/>
       </xacro:range_sensor>
-      <xacro:range_sensor name="${name}_sonar_02" parent="${name}" ros_topic="sonar_${name}" update_rate="5" maxRange="1.0" minRange="0.02" fov="0.5" radiation="ultrasound">
-        <origin xyz="-0.259 0.0 0.173" rpy="0 0 ${180 * deg_to_rad}"/>
+      <xacro:range_sensor name="${name}_sonar_02" parent="${name}" ros_topic="sonar4_${name}" update_rate="1" maxRange="3.0" minRange="0.02" fov="0.5" radiation="ultrasound">
+        <origin xyz="${0.259*cos(30*deg_to_rad)} ${0.259*sin(30*deg_to_rad)}  0.173" rpy="0 0 ${30*deg_to_rad}"/>
       </xacro:range_sensor>
-      <xacro:range_sensor name="${name}_sonar_01" parent="${name}" ros_topic="sonar_${name}" update_rate="5" maxRange="1.0" minRange="0.02" fov="0.5" radiation="ultrasound">
-        <origin xyz="-0.183 -0.183 0.173" rpy="0 0 ${225 * deg_to_rad}"/>
+      <xacro:range_sensor name="${name}_sonar_03" parent="${name}" ros_topic="sonar4_${name}" update_rate="1" maxRange="3.0" minRange="0.02" fov="0.5" radiation="ultrasound">
+        <origin xyz="${0.259*cos(60*deg_to_rad)} ${0.259*sin(60*deg_to_rad)}  0.173" rpy="0 0 ${60*deg_to_rad}"/>
+      </xacro:range_sensor>
+      <xacro:range_sensor name="${name}_sonar_04" parent="${name}" ros_topic="sonar4_${name}" update_rate="1" maxRange="3.0" minRange="0.02" fov="0.5" radiation="ultrasound">
+        <origin xyz="${0.259*cos(90*deg_to_rad)} ${0.259*sin(90*deg_to_rad)}  0.173" rpy="0 0 ${90*deg_to_rad}"/>
+      </xacro:range_sensor>
+      <xacro:range_sensor name="${name}_sonar_05" parent="${name}" ros_topic="sonar4_${name}" update_rate="1" maxRange="3.0" minRange="0.02" fov="0.5" radiation="ultrasound">
+        <origin xyz="${0.259*cos(120*deg_to_rad)} ${0.259*sin(120*deg_to_rad)}  0.173" rpy="0 0 ${120*deg_to_rad}"/>
+      </xacro:range_sensor>
+      <xacro:range_sensor name="${name}_sonar_06" parent="${name}" ros_topic="sonar4_${name}" update_rate="1" maxRange="3.0" minRange="0.02" fov="0.5" radiation="ultrasound">
+        <origin xyz="${0.259*cos(150*deg_to_rad)} ${0.259*sin(150*deg_to_rad)}  0.173" rpy="0 0 ${150*deg_to_rad}"/>
+      </xacro:range_sensor>
+      <xacro:range_sensor name="${name}_sonar_07" parent="${name}" ros_topic="sonar4_${name}" update_rate="1" maxRange="3.0" minRange="0.02" fov="0.5" radiation="ultrasound">
+        <origin xyz="${0.259*cos(180*deg_to_rad)} ${0.259*sin(180*deg_to_rad)}  0.173" rpy="0 0 ${180*deg_to_rad}"/>
+      </xacro:range_sensor>
+      <xacro:range_sensor name="${name}_sonar_08" parent="${name}" ros_topic="sonar4_${name}" update_rate="1" maxRange="3.0" minRange="0.02" fov="0.5" radiation="ultrasound">
+        <origin xyz="${0.259*cos(210*deg_to_rad)} ${0.259*sin(210*deg_to_rad)}  0.173" rpy="0 0 ${210*deg_to_rad}"/>
+      </xacro:range_sensor>
+      <xacro:range_sensor name="${name}_sonar_09" parent="${name}" ros_topic="sonar4_${name}" update_rate="1" maxRange="3.0" minRange="0.02" fov="0.5" radiation="ultrasound">
+        <origin xyz="${0.259*cos(240*deg_to_rad)} ${0.259*sin(240*deg_to_rad)}  0.173" rpy="0 0 ${240*deg_to_rad}"/>
+      </xacro:range_sensor>
+      <xacro:range_sensor name="${name}_sonar_10" parent="${name}" ros_topic="sonar4_${name}" update_rate="1" maxRange="3.0" minRange="0.02" fov="0.5" radiation="ultrasound">
+        <origin xyz="${0.259*cos(270*deg_to_rad)} ${0.259*sin(270*deg_to_rad)}  0.173" rpy="0 0 ${270*deg_to_rad}"/>
+      </xacro:range_sensor>
+      <xacro:range_sensor name="${name}_sonar_11" parent="${name}" ros_topic="sonar4_${name}" update_rate="1" maxRange="3.0" minRange="0.02" fov="0.5" radiation="ultrasound">
+        <origin xyz="${0.259*cos(300*deg_to_rad)} ${0.259*sin(300*deg_to_rad)}  0.173" rpy="0 0 ${300*deg_to_rad}"/>
+      </xacro:range_sensor>
+      <xacro:range_sensor name="${name}_sonar_12" parent="${name}" ros_topic="sonar4_${name}" update_rate="1" maxRange="3.0" minRange="0.02" fov="0.5" radiation="ultrasound">
+        <origin xyz="${0.259*cos(330*deg_to_rad)} ${0.259*sin(330*deg_to_rad)}  0.173" rpy="0 0 ${330*deg_to_rad}"/>
       </xacro:range_sensor>
     </xacro:if>

File: environment_pkg/urdf/tiago.urdf.xacro (robot description, xacro)
@@ -72,15 +72,5 @@
   <xacro:include filename="$(find pal_urdf_utils)/urdf/deg_to_rad.xacro" />
   <!-- Base -->
-  <xacro:include filename="$(find ${base_type}_description)/urdf/base/base_sensors.urdf.xacro" />
-  <xacro:include filename="$(find hector_sensors_description)/urdf/sonar_sensor.urdf.xacro"/>
-  <xacro:sonar_sensor name="base_sonar1" parent="base_link" ros_topic="base_sonar1" update_rate="10.0" min_range="0.2" max_range="3.5" field_of_view="0.785398" ray_count="5">
-    <origin xyz="0.0 0.0 0.0" rpy="0 0 0"/>
-  </xacro:sonar_sensor>
-  <xacro:sonar_sensor name="base_sonar2" parent="base_link" ros_topic="base_sonar2" update_rate="10.0" min_range="-0.2" max_range="-3.5" field_of_view="0.785398" ray_count="5">
-    <origin xyz="0.0 0.0 0.0" rpy="0 0 0"/>
-  </xacro:sonar_sensor>
-  <xacro:sonar_sensor name="base_sonar3" parent="base_link" ros_topic="base_sonar3" update_rate="10.0" min_range="0.2" max_range="3.5" field_of_view="0.785398" ray_count="5">
-    <origin xyz="0.0 0.0 0.0" rpy="0 0 0"/>
-  </xacro:sonar_sensor>
+  <xacro:include filename="$(find environment_pkg)/urdf/base_sensors.urdf.xacro" />
   <!-- Torso -->
   <xacro:include filename="$(find tiago_description)/urdf/torso/torso.urdf.xacro" />
